Commit message: Add forward kinematics

File: config/example.urdf (robot description, URDF)
Before this commit: robot crichton, 43 links, 42 joints
Joints:
- joint crichton_left_1_joint: origin xyz=0 0.12 0 rpy=1.57 3.1416 0 -> xyz=0 0.12 0 rpy=1.5707963265 3.141592653 0
- joint crichton_left_2_joint: origin xyz=0 0 -0.18 rpy=-1.57 0 0 -> xyz=0 0 -0.18 rpy=-1.5707963265 0 0
- joint crichton_left_3_joint: origin xyz=0 0 0 rpy=1.57 0 0 -> xyz=0 0 0 rpy=1.5707963265 0 0
- joint crichton_left_4_joint: origin xyz=0 0 -0.328 rpy=-1.57 0 0 -> xyz=0 0 -0.328 rpy=-1.5707963265 0 0
- joint crichton_left_5_joint: origin xyz=0 0 0 rpy=1.57 0 0 -> xyz=0 0 0 rpy=1.5707963265 0 0
- joint crichton_left_6_joint: origin xyz=0 0 -0.323 rpy=1.57 0 0 -> xyz=0 0 -0.323 rpy=1.5707963265 0 0
- joint crichton_left_7_joint: origin xyz=0 -0.1672 0 rpy=-1.57 0 0 -> xyz=0 -0.1672 0 rpy=-1.5707963265 0 0
- joint crichton_left_thumb_1_joint: origin xyz=0 0.03811 0.0745  rpy=0 0 -1.5708 -> xyz=0 0.03811 0.0745  rpy=0 0 -1.5707963265
- joint crichton_right_1_joint: origin xyz=0 0.12 0 rpy=1.57 3.1416 0 -> xyz=0 0.12 0 rpy=1.5707963265 3.141592653 0
- joint crichton_right_2_joint: origin xyz=0 0 -0.18 rpy=-1.57 0 0 -> xyz=0 0 -0.18 rpy=-1.5707963265 0 0
- joint crichton_right_3_joint: origin xyz=0 0 0 rpy=1.57 0 0 -> xyz=0 0 0 rpy=1.5707963265 0 0
- joint crichton_right_4_joint: origin xyz=0 0 -0.328 rpy=-1.57 0 0 -> xyz=0 0 -0.328 rpy=-1.5707963265 0 0
- joint crichton_right_5_joint: origin xyz=0 0 0 rpy=1.57 0 0 -> xyz=0 0 0 rpy=1.5707963265 0 0
- joint crichton_right_6_joint: origin xyz=0 0 -0.323 rpy=1.57 0 0 -> xyz=0 0 -0.323 rpy=1.5707963265 0 0
- joint crichton_right_7_joint: origin xyz=0 -0.1672 0 rpy=-1.57 0 0 -> xyz=0 -0.1672 0 rpy=-1.5707963265 0 0
- joint crichton_right_thumb_1_joint: origin xyz=0 0.03811 0.0745  rpy=0 0 -1.5708 -> xyz=0 0.03811 0.0745  rpy=0 0 -1.5707963265
